File: kicad/kicad.kicad_pcb (KiCad board)
At the start: 2 copper layers, 138.4 x 85.1 mm, 27 parts, among them U1 ESP32-DEVKITC-32D

Commit message: Zwischenstand
Parts:
- removed 5VDown1: LM2596S, ft-playground:LM2596S
- removed VarDownF1, VarUpF1: Fuse, Fuse:Fuse_BelFuse_0ZRE0125FF_L21.2mm_W5.3mm
- added Ethernet1: RJ45, Connector_RJ:RJ45_Amphenol_54602-x08_Horizontal, F.Cu at (12.7, 49.5)
- added POE1: RJ45, Connector_RJ:RJ45_Amphenol_54602-x08_Horizontal, F.Cu at (12.7, 67.3)
- added U2: ESP32-DEVKITC-32D, ft-playground:MODULE_ESP32-DEVKITC-32D, F.Cu at (-66.0, 65.4)
- Bat1VC1: footprint Capacitor_THT:C_Axial_L3.8mm_D2.6mm_P7.50mm_Horizontal -> Capacitor_SMD:C_1806_4516Metric_Pad1.57x1.80mm_HandSolder
- Bat1VRG1, Bat1VRS1: footprint Resistor_THT:R_Axial_DIN0207_L6.3mm_D2.5mm_P15.24mm_Horizontal -> Resistor_SMD:R_1210_3225Metric_Pad1.42x2.65mm_HandSolder
- Bat2VC1, DownVC1, UpVC1: footprint Capacitor_THT:C_Axial_L3.8mm_D2.6mm_P7.50mm_Horizontal -> Capacitor_SMD:C_1806_4516Metric_Pad1.57x1.80mm_HandSolder; moved to B.Cu
- Bat2VRG1, Bat2VRS1, DownVRG1, DownVRS1, UpVRG1, UpVRS1: footprint Resistor_THT:R_Axial_DIN0207_L6.3mm_D2.5mm_P15.24mm_Horizontal -> Resistor_SMD:R_1210_3225Metric_Pad1.42x2.65mm_HandSolder; moved to B.Cu
- ESP32PWRSRC1: footprint TerminalBlock:TerminalBlock_bornier-2_P5.08mm -> Connector_PinHeader_2.54mm:PinHeader_1x02_P2.54mm_Vertical
- F1, F2: footprint Fuse:Fuse_BelFuse_0ZRE0125FF_L21.2mm_W5.3mm -> Fuse:Fuse_Bourns_MF-RG400
- U1: value ESP32-DEVKITC-32D -> D36V6F3; footprint ft-playground:MODULE_ESP32-DEVKITC-32D -> ft-playground:D36V6F3
- moved Bat2 181.8 mm to (-30.5, 100.7), turned to 90 degrees
- moved VarStepUp1 146.7 mm to (-45.7, 38.7)
- moved F2 139.4 mm to (-19.1, 101.0), turned to 270 degrees
- moved Out:Down1 139.4 mm to (13.3, 92.7), turned to 180 degrees
- moved Out:Up1 139.2 mm to (13.3, 79.4), turned to 180 degrees
- moved Bat1 135.7 mm to (14.6, 101.0), turned to 90 degrees
- moved Bat2VRS1 129.2 mm to (-41.3, 102.9)
- moved Bat1VRS1 128.4 mm to (-41.3, 102.9)
- moved Bat2VC1 124.7 mm to (-41.3, 90.8)
- moved D2 123.3 mm to (-11.4, 105.4)
- moved UpVRS1 114.8 mm to (-9.74, 42.5), turned to 0 degrees
- moved DownVRS1 114.3 mm to (-2.54, 88.9), turned to 0 degrees
- moved F1 113.8 mm to (5.71, 106.7), turned to 90 degrees
- moved D1 111.9 mm to (-1.27, 105.4), turned to 90 degrees
- moved UpVRG1 110.6 mm to (-9.53, 49.5), turned to 180 degrees
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Connections:
- ESP32PWRSRC1 pad 2: Net-(5VDown1-Pad1) -> Net-(ESP32PWRSRC1-Pad2)
- Out:Down1 pad 1: Net-(Out:Down1-Pad1) -> Net-(DownVRS1-Pad2)
- U1 pad 2: (no net) -> +12V
- U1 pad 3: (no net) -> GND
- U1 pad 4: (no net) -> Net-(ESP32PWRSRC1-Pad2)
- UpVC1 pad 1: Net-(U1-Pad7) -> Net-(U2-Pad8)
- UpVRG1 pad 2: Net-(U1-Pad7) -> Net-(U2-Pad8)
- UpVRS1 pad 1: Net-(U1-Pad7) -> Net-(U2-Pad8)
- VarStepUp1 pad 1: Net-(VarStepUp1-Pad1) -> +24V
Routing:
- net GND: track 197.3 -> 360.9 mm
- net Net-(5VDown1-Pad1): track 144.9 -> 0.00 mm
- net Net-(U1-Pad7): track 100.3 -> 0.00 mm
- net Net-(Bat2VC1-Pad1): track 125.9 -> 41.8 mm
- net +12V: track 170.6 -> 100.3 mm
- net Net-(Bat1VC1-Pad1): track 104.1 -> 41.5 mm
- net Net-(U2-Pad8): track 0.00 -> 60.2 mm
- net Net-(DownVC1-Pad1): track 111.0 -> 64.6 mm
- net Net-(VarStepUp1-Pad1): track 45.9 -> 0.00 mm
- net Net-(Bat1VRS1-Pad2): track 17.6 -> 52.3 mm
- net Net-(Ethernet1-Pad1): track 0.00 -> 30.2 mm
- net Net-(Ethernet1-Pad2): track 0.00 -> 28.8 mm
- net Net-(Ethernet1-Pad6): track 0.00 -> 26.1 mm
- net Net-(Out:Down1-Pad1): track 23.0 -> 0.00 mm
- net Net-(Ethernet1-Pad3): track 0.00 -> 20.5 mm
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- removed copper zone on B.Cu, net GND
Other:
- board size 138.4 x 85.1 mm -> 76.8 x 74.3 mm
