File: kicad/kicad.sch (KiCad schematic (older format))
At the start: 14 parts, among them J1 Jack-DC, U1 ESP32-DEVKITC-32D, U3 D36V6F3, U4 xL6019

Commit message: Update
Parts:
- removed U3: D36V6F3, symbol D36V6F3:D36V6F3
- added F1, F2: Fuse, symbol Device:Fuse
- added J2: Jack-DC, symbol Connector:Jack-DC
- added J3, J4, J5: USB_A, symbol Connector:USB_A
- added U2: D24V50F5, symbol D36V6F3:D24V50F5
Connections:
- net GND: now also J2.2, J3.4 (GND), J4.4 (GND), J5.4 (GND), U2.3 (GND), U2.4 (GND)
- net +5V: now reaches U1.19 (EXT_5V)
- net +5V: now also J3.1 (VBUS), J4.1 (VBUS), J5.1 (VBUS), U2.5 (VOUT)
- net +15V: now reaches R2.2, U4.2 (VIN)
- net +15V: now also F1.1, F2.1, J2.1, U2.2 (VIN); no longer D1.2 (A), D2.2 (A)
- new net: D1.2 (A), F1.2
- new net: D2.2 (A), F2.2
- no-connect marks 34 -> 44
Other:
- moved on the sheet: BT1, BT2, C1, C2, D1, D2, J1, R1, R2, R3, R4, U1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

Commit message: Remaining components
Parts:
- removed J4, J5: USB_A, symbol Connector:USB_A
- removed U2: D24V50F5, symbol D36V6F3:D24V50F5
- added C4, C5: CP, symbol Device:CP
- added F3, F4, F5: Fuse, symbol Device:Fuse
- added J4, J5: RJ45, symbol Connector:RJ45
- added J6, J7: Jack-DC, symbol Connector:Jack-DC
- added JP1: Jumper, symbol Device:Jumper
- added R10, R5, R7, R9: R, symbol Device:R
- added U2, U3: LM2596S, symbol XL60919:LM2596S
Connections:
- net +5V: now also J1.1, F4.2; no longer U1.19 (EXT_5V)
- net GND: now also U1.26 (GND2), C4.2, C5.2, J4.7, J4.8, J6.2, J7.2, R7.1, R9.1, U2.3 (GND), U2.4 (GND), U3.3 (GND), U3.4 (GND)
- net at U1.5 (IO34): now also C1.1, R1.2, R2.1
- net at U1.6 (IO35): now also C2.1, R3.2, R4.1
- net at D1.1 (K): now also F1.1, R2.2; no longer BT1.1 (+)
- net at F1.2: now also BT1.1 (+); no longer D1.2 (A)
- net at D2.1 (K): now also F2.1, R4.2; no longer BT2.1 (+)
- net at F2.2: now also BT2.1 (+); no longer D2.2 (A)
- removed net +15V: F1.1, F2.1, J2.1, R2.2, U4.2 (VIN)
- new net: JP1.1, U1.19 (EXT_5V)
- new net: C4.1, R5.1, R7.2, U1.7 (IO32)
- new net: C5.1, R10.1, R9.2, U1.8 (IO33)
- new net: F3.1, R10.2, U2.1 (VOUT)
- new net: F4.1, JP1.2, U3.1 (VOUT)
- new net: F3.2, J2.1
- new net: F5.2, U4.1 (VOUT)
- new net: J4.1, J5.1
- new net: J4.2, J5.2
- new net: J4.3, J5.3
- new net: J4.6, J5.6
- new net +12V: D1.2 (A), D2.2 (A), J7.1, U2.2 (VIN), U3.2 (VIN), U4.2 (VIN)
- new net +24V: F5.1, J4.4, J4.5, J6.1, R5.2
- no-connect marks 44 -> 38
Other:
- moved on the sheet: BT1, BT2, C1, D1, D2, J1, J2, J3, R1, U1

Commit message: Zwischenstand 2020-12-25
Parts:
- removed F4: Fuse, symbol Device:Fuse
- removed J1, J7: Jack-DC, symbol Connector:Jack-DC
- removed J3: USB_A, symbol Connector:USB_A
- removed J4, J5: RJ45, symbol Connector:RJ45
- 5VDown1: renamed from U3; footprint (none) -> ft-playground:LM2596S
- Bat1: renamed from BT1; footprint (none) -> Connector_BarrelJack:BarrelJack_Horizontal
- Bat1VC1: renamed from C1; footprint (none) -> Capacitor_THT:C_Axial_L3.8mm_D2.6mm_P7.50mm_Horizontal
- Bat1VRG1: renamed from R1; footprint (none) -> Resistor_THT:R_Axial_DIN0207_L6.3mm_D2.5mm_P15.24mm_Horizontal
- Bat1VRS1: renamed from R2; footprint (none) -> Resistor_THT:R_Axial_DIN0207_L6.3mm_D2.5mm_P15.24mm_Horizontal
- Bat2: renamed from BT2; footprint (none) -> Connector_BarrelJack:BarrelJack_Horizontal
- Bat2VC1: renamed from C2; footprint (none) -> Capacitor_THT:C_Axial_L3.8mm_D2.6mm_P7.50mm_Horizontal
- Bat2VRG1: renamed from R3; footprint (none) -> Resistor_THT:R_Axial_DIN0207_L6.3mm_D2.5mm_P15.24mm_Horizontal
- Bat2VRS1: renamed from R4; footprint (none) -> Resistor_THT:R_Axial_DIN0207_L6.3mm_D2.5mm_P15.24mm_Horizontal
- D1, D2: footprint (none) -> Diode_THT:D_DO-15_P5.08mm_Vertical_AnodeUp
- DownVC1: renamed from C5; footprint (none) -> Capacitor_THT:C_Axial_L3.8mm_D2.6mm_P7.50mm_Horizontal
- DownVRG1: renamed from R9; footprint (none) -> Resistor_THT:R_Axial_DIN0207_L6.3mm_D2.5mm_P15.24mm_Horizontal
- DownVRS1: renamed from R10; footprint (none) -> Resistor_THT:R_Axial_DIN0207_L6.3mm_D2.5mm_P15.24mm_Horizontal
- ESP32PWRSRC1: renamed from JP1; footprint (none) -> TerminalBlock:TerminalBlock_bornier-2_P5.08mm
- F1, F2: footprint (none) -> Fuse:Fuse_BelFuse_0ZRE0125FF_L21.2mm_W5.3mm
- Out:Down1: renamed from J2; footprint (none) -> Connector_BarrelJack:BarrelJack_Horizontal
- Out:Up1: renamed from J6; footprint (none) -> Connector_BarrelJack:BarrelJack_Horizontal
- U1: footprint MODULE_ESP32-DEVKITC-32D -> ft-playground:MODULE_ESP32-DEVKITC-32D
- UpVC1: renamed from C4; footprint (none) -> Capacitor_THT:C_Axial_L3.8mm_D2.6mm_P7.50mm_Horizontal
- UpVRG1: renamed from R7; footprint (none) -> Resistor_THT:R_Axial_DIN0207_L6.3mm_D2.5mm_P15.24mm_Horizontal
- UpVRS1: renamed from R5; footprint (none) -> Resistor_THT:R_Axial_DIN0207_L6.3mm_D2.5mm_P15.24mm_Horizontal
- VarDownF1: renamed from F3; footprint (none) -> Fuse:Fuse_BelFuse_0ZRE0125FF_L21.2mm_W5.3mm
- VarStepDown1: renamed from U2; footprint (none) -> ft-playground:LM2596S
- VarStepUp1: renamed from U4; footprint (none) -> ft-playground:XL6019
- VarUpF1: renamed from F5; footprint (none) -> Fuse:Fuse_BelFuse_0ZRE0125FF_L21.2mm_W5.3mm
Connections:
- net GND: now also VarStepUp1.3 (GND), VarStepUp1.4 (GND)
- no-connect marks 38 -> 31
Other:
- moved on the sheet: Bat1VC1, Bat1VRG1, Bat2VC1, Bat2VRG1, DownVC1, ESP32PWRSRC1, Out:Up1, UpVRG1

Commit message: Zwischenstand
Parts:
- removed 5VDown1: LM2596S, ft-playground:LM2596S, symbol XL60919:LM2596S
- removed VarDownF1, VarUpF1: Fuse, Fuse:Fuse_BelFuse_0ZRE0125FF_L21.2mm_W5.3mm, symbol Device:Fuse
- added Ethernet, POE: RJ45, Connector_RJ:RJ45_Amphenol_54602-x08_Horizontal, symbol Connector:RJ45
- added U1: D36V6F3, ft-playground:D36V6F3, symbol D36V6F3:D36V6F3
- Bat1VC1, Bat2VC1, DownVC1, UpVC1: footprint Capacitor_THT:C_Axial_L3.8mm_D2.6mm_P7.50mm_Horizontal -> Capacitor_SMD:C_1806_4516Metric_Pad1.57x1.80mm_HandSolder
- Bat1VRG1, Bat1VRS1, Bat2VRG1, Bat2VRS1, DownVRG1, DownVRS1, UpVRG1, UpVRS1: footprint Resistor_THT:R_Axial_DIN0207_L6.3mm_D2.5mm_P15.24mm_Horizontal -> Resistor_SMD:R_1210_3225Metric_Pad1.42x2.65mm_HandSolder
- ESP32PWRSRC1: footprint TerminalBlock:TerminalBlock_bornier-2_P5.08mm -> Connector_PinHeader_2.54mm:PinHeader_1x02_P2.54mm_Vertical
- F1, F2: footprint Fuse:Fuse_BelFuse_0ZRE0125FF_L21.2mm_W5.3mm -> Fuse:Fuse_Bourns_MF-RG400
- renumbered U1 to U2
Connections:
- net +12V: now also U1.2 (VIN)
- net +24V: now also VarStepUp1.1 (VOUT), POE.4, POE.5
- net GND: now also POE.7, POE.8, U1.3 (GND); no longer U2.26 (GND2)
- net at U2.1 (3V3): now also ESP32PWRSRC1.1
- net at U2.19 (EXT_5V): no longer ESP32PWRSRC1.1
- net at UpVC1.1, UpVRG1.2, UpVRS1.1: now also U2.8 (IO33); no longer U2.7 (IO32)
- net at DownVC1.1, DownVRG1.2, DownVRS1.1: now also U2.7 (IO32); no longer U2.8 (IO33)
- net at DownVRS1.2, VarStepDown1.1 (VOUT): now also Out:Down1.1
- net at ESP32PWRSRC1.2: now also U1.4 (VOUT)
- new net: Ethernet.1, POE.1
- new net: Ethernet.2, POE.2
- new net: Ethernet.3, POE.3
- new net: Ethernet.6, POE.6
- no-connect marks 31 -> 38

Commit message: schem: Improve layout & Re-Annotate the schematics
Parts:
- removed Bat1VC1, Bat2VC1, DownVC1, UpVC1: CP, Capacitor_SMD:C_1806_4516Metric_Pad1.57x1.80mm_HandSolder, symbol Device:CP
- removed Bat1VRG1, Bat1VRS1, Bat2VRG1, Bat2VRS1, DownVRG1, DownVRS1, UpVRG1, UpVRS1: R, Resistor_SMD:R_1210_3225Metric_Pad1.42x2.65mm_HandSolder, symbol Device:R
- removed D1, D2: DIODE, Diode_THT:D_DO-15_P5.08mm_Vertical_AnodeUp, symbol pspice:DIODE
- removed ESP32PWRSRC1: Jumper, Connector_PinHeader_2.54mm:PinHeader_1x02_P2.54mm_Vertical, symbol Device:Jumper
- removed Out:Down1, Out:Up1: Jack-DC, Connector_BarrelJack:BarrelJack_Horizontal, symbol Connector:Jack-DC
- added C1, C2, C3, C4, C5: CP, symbol Device:CP
- added D1, D2: D, symbol Device:D
- added J2, J4: Barrel_Jack, symbol Connector:Barrel_Jack
- added JP1: Jumper, symbol Device:Jumper
- added R1, R10, R2, R3, R4, R5, R6, R7, R8, R9: R, symbol Device:R
- Bat1, Bat2: footprint Connector_BarrelJack:BarrelJack_Horizontal -> (none)
- F1, F2: footprint Fuse:Fuse_Bourns_MF-RG400 -> (none)
- U3: renamed from U1; footprint ft-playground:D36V6F3 -> (none)
- renumbered Ethernet to J1, POE to J3, U2 to U1, VarStepUp1 to U2, VarStepDown1 to U4
Connections:
- net labels added: 12V_BAT, 24V, 24V_SENSE, 3V3, 3V3_SENSE, BAT1_SENSE, BAT2_SENSE, xxV, xxV_SENSE
- net labels removed: +12V, +24V
- wire segments 95 -> 99
- no-connect marks 38 -> 37
Other:
- note added: "Connectors"
- note added: "Input Protection & Sensing"
- note added: "Microcontroller"
- note added: "TODO:\n- Find correct resistor values\n- Find correct capacitor values\n- Check if ESP32 nreed more than one GND connection"
- note added: "Voltage Regulation"
- moved on the sheet: J1, J3, U1, U2, U3, U4
